File: copy/copy.kicad_pcb (KiCad board)
At the start: 2 copper layers, 263.2 x 132.1 mm, 121 parts, among them J1 Conn_02x07_Row_Letter_Last, J10 Conn_02x07_Row_Letter_Last, J11 Conn_01x03_Pin, J2 01x02, J3 Barrel_Jack_Switch, J4 PINHD_1x2_Female, J5 Conn_01x03_Pin, J6 Conn_02x07_Row_Letter_Last, J7 Conn_01x03_Pin, J8 Conn_02x07_Row_Letter_Last, J9 Conn_01x03_Pin, Q1 TO-220*3_HS_inverter_type, Q14 TO-220*3_HS_inverter_type, Q15 TO-220*3_HS_inverter_type, Q2 TO-220*3_HS_inverter_type, T1 Transformer_1P_1S, U1 LM741, U2 Opamp_Dual, U3 BluePill, U6 L7805, U7 AMS1117-3.3, U8 ACS712xLCTR-05B

Commit message: complete
Parts:
- R43, R44: value 470E -> 1K
- moved D9 7.66 mm to (159.8, 120.9), turned to 90 degrees
Connections:
- D9 pad 1: Net-(D9-K) -> CutOff
- D9 pad 2: CutOff -> Net-(D9-A)
- R43 pad 1: Net-(D9-K) -> Net-(D9-A)
- U2 pad 7: Net-(D9-K) -> Net-(D9-A)
Routing:
- net Net-(D9-K): track 6.66 -> 0.00 mm
- net Net-(D9-A): track 0.00 -> 6.66 mm
