File: copy/untitled.kicad_sch (KiCad schematic)
At the start: 11 parts, among them U2 Opamp_Dual

Commit message: complete
Parts:
- R43, R44: value 470E -> 1K
Connections:
- net CMP_Out: now also D9.1 (K); no longer D9.2 (A)
- net at R43.1, U2.7: now also D9.2 (A); no longer D9.1 (K)
Other:
- moved on the sheet: D9
Changed lines of the file:
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@@
 		)
 		(property "Value" "5V"
-			(at 173.99 77.47 0)
-			(effects
-				(font
-					(size 1.27 1.27)
-				)
+			(at 176.53 81.2799 0)
+			(effects
+				(font
+					(size 1.27 1.27)
+				)
+				(justify left)
 			)
 		)
@@
 			)
 		)
-		(property "Value" "470E"
+		(property "Value" "1K"
 			(at 176.53 91.4399 90)
 			(effects
@@
 			)
 		)
-		(property "Value" "470E"
+		(property "Value" "1K"
 			(at 166.37 121.9199 90)
 			(effects
@@
 		)
 		(property "Value" "5V"
-			(at 163.83 107.95 0)
-			(effects
-				(font
-					(size 1.27 1.27)
-				)
+			(at 166.37 111.7599 0)
+			(effects
+				(font
+					(size 1.27 1.27)
+				)
+				(justify left)
 			)
 		)
@@
 	(symbol
 		(lib_id "Device:D")
-		(at 173.99 116.84 90)
+		(at 173.99 116.84 270)
 		(unit 1)
 		(exclude_from_sim no)
@@
 					(size 1.27 1.27)
 				)
-				(justify right)
+				(justify left)
 			)
 		)
@@
 					(size 1.27 1.27)
 				)
-				(justify right)
-			)
-		)
+				(justify left)
+			)
+		)
